File: AK4458VN_breakout/AK4458VN_breakout.kicad_pcb (KiCad board)
At the start: 2 copper layers, 50 x 73.2 mm, 83 parts, among them J1 Conn_02x18_Odd_Even, U1 AK4458VN, U4 NE5532DR, U5 NE5532DR, U6 NE5532DR, U7 NE5532DR

Commit message: ak4458vn breakout v1.1
Parts:
- added C30: 0.1u, Capacitor_SMD:C_0603_1608Metric, F.Cu at (129.2, 69.4)
- added C31: 0.1u, Capacitor_SMD:C_0603_1608Metric, F.Cu at (120.8, 69.4)
Connections:
- J1 pad 1: DVSS -> VDD18
- J1 pad 10: LRCK/DSDL1 -> SDTI1/DSDR1
- J1 pad 12: SDTI1/DSDR1 -> SDTI2/DSDL2
- J1 pad 14: SDTI2/DSDL2 -> SDTI3/DSDR2/TDMO1
- J1 pad 16: SDTI3/DSDR2/TDMO1 -> VREFH
- J1 pad 2: VDD18 -> PDN
- J1 pad 22: SDTI4/DSDL3/TDMO2 -> VREFL
- J1 pad 24: DSDR3 -> SDTI4/DSDL3/TDMO2
- J1 pad 26: DSDL4 -> DSDR3
- J1 pad 27: unconnected-(J1-Pin_27-Pad27) -> V12P
- J1 pad 28: DSDR4 -> DSDL4
- J1 pad 29: V12P -> I2C
- J1 pad 3: TVDD -> DVSS
- J1 pad 30: DZF/SMUTE -> DSDR4
- J1 pad 31: I2C -> PS/CAD0_SPI
- J1 pad 32: CAD1/DCHAIN -> DZF/SMUTE
- J1 pad 33: PS/CAD0_SPI -> CAD0_I2C/CSN/_DIF
- J1 pad 34: SDA/CDTI/TDM0 -> CAD1/DCHAIN
- J1 pad 35: CAD0_I2C/CSN/_DIF -> SCL/CCLK/TDM1
- J1 pad 36: SCL/CCLK/TDM1 -> SDA/CDTI/TDM0
- J1 pad 4: PDN -> MCLK
- J1 pad 5: LDOE -> TVDD
- J1 pad 6: MCLK -> BICK/DCLK
- J1 pad 7: V12N -> LDOE
- J1 pad 8: BICK/DCLK -> LRCK/DSDL1
- J1 pad 9: unconnected-(J1-Pin_9-Pad9) -> V12N
Routing:
- net VDD18: track 78.0 -> 87.8 mm, vias 2 -> 3
- net TVDD: track 97.8 -> 89.2 mm
- net VREFH: track 50.3 -> 57.9 mm
- net I2C: track 28.1 -> 22.1 mm
- net AVSS: track 46.9 -> 41.0 mm, vias 84 -> 85
- net VREFL: track 43.2 -> 49.1 mm
- net LDOE: track 27.5 -> 21.9 mm
- net SCL/CCLK/TDM1: track 21.0 -> 25.4 mm
- net SDTI3/DSDR2/TDMO1: track 7.05 -> 10.4 mm
- net SDTI4/DSDL3/TDMO2: track 7.03 -> 10.3 mm
- net PDN: track 18.2 -> 20.8 mm
- net DZF/SMUTE: track 14.3 -> 16.9 mm
- net BICK/DCLK: track 14.6 -> 17.2 mm
- net DSDR4: track 12.3 -> 14.9 mm
- net SDA/CDTI/TDM0: track 18.2 -> 20.7 mm
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Other:
- board text added: "AK4458 Breakout Rev 1.1 Daniel Lewis daniel.lewis.software.engineer@gmail.com Alex Sludds alexsludds@gmail.com"
