File: AK4458VN_breakout/AK4458VN_breakout.kicad_sch (KiCad schematic)
At the start: 83 parts, among them J1 Conn_02x18_Odd_Even, U1 AK4458VN, U4 NE5532DR, U5 NE5532DR, U6 NE5532DR, U7 NE5532DR

Commit message: ak4458vn breakout v1.1
Parts:
- added C30, C31: 0.1u, Capacitor_SMD:C_0603_1608Metric, symbol Device:C
Connections:
- net BICK/DCLK: now also J1.6 (Pin_6); no longer J1.8 (Pin_8)
- net CAD0_I2C/CSN/_DIF: now also J1.33 (Pin_33); no longer J1.35 (Pin_35)
- net CAD1/DCHAIN: now also J1.34 (Pin_34); no longer J1.32 (Pin_32)
- net DSDL4: now also J1.28 (Pin_28); no longer J1.26 (Pin_26)
- net DSDR3: now also J1.26 (Pin_26); no longer J1.24 (Pin_24)
- net DSDR4: now also J1.30 (Pin_30); no longer J1.28 (Pin_28)
- net DVSS: now also J1.3 (Pin_3); no longer J1.1 (Pin_1)
- net DZF/SMUTE: now also J1.32 (Pin_32); no longer J1.30 (Pin_30)
- net I2C: now also J1.29 (Pin_29); no longer J1.31 (Pin_31)
- net LDOE: now also J1.7 (Pin_7); no longer J1.5 (Pin_5)
- net LRCK/DSDL1: now also J1.8 (Pin_8); no longer J1.10 (Pin_10)
- net MCLK: now also J1.4 (Pin_4); no longer J1.6 (Pin_6)
- net PDN: now also J1.2 (Pin_2); no longer J1.4 (Pin_4)
- net PS/CAD0_SPI: now also J1.31 (Pin_31); no longer J1.33 (Pin_33)
- net SCL/CCLK/TDM1: now also J1.35 (Pin_35); no longer J1.36 (Pin_36)
- net SDA/CDTI/TDM0: now also J1.36 (Pin_36); no longer J1.34 (Pin_34)
- net SDTI1/DSDR1: now also J1.10 (Pin_10); no longer J1.12 (Pin_12)
- net SDTI2/DSDL2: now also J1.12 (Pin_12); no longer J1.14 (Pin_14)
- net SDTI3/DSDR2/TDMO1: now also J1.14 (Pin_14); no longer J1.16 (Pin_16)
- net SDTI4/DSDL3/TDMO2: now also J1.24 (Pin_24); no longer J1.22 (Pin_22)
- net TVDD: now also J1.5 (Pin_5); no longer J1.3 (Pin_3)
- net V12N: now also J1.9 (Pin_9); no longer J1.7 (Pin_7)
- net V12P: now also J1.27 (Pin_27); no longer J1.29 (Pin_29)
- net VDD18: now also J1.1 (Pin_1); no longer J1.2 (Pin_2)
- net VREFH: now also J1.16 (Pin_16), C30.1, C31.1
- net VREFL: now also J1.22 (Pin_22), C30.2, C31.2
