File: teensy_dc_interface/teensy_dc_interface.kicad_pcb (KiCad board)
At the start: 2 copper layers, 80.9 x 128.5 mm, 165 parts, among them J1 Chan 1 Out, J10 3.5mm_Mono_Switched_SymSmall_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, J11 Conn_01x03, J12 Conn_01x03, J13 Conn_01x03, J2 Chan 2 Out, J3 Chan 3 Out, J4 Chan 4 Out, J5 Chan 5 Out, J6 Chan 6 Out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

Commit message: mounting holes
Parts:
- added H2: MountingHole, 4ms_Faceplate:Faceplate_Rail_Mount_Slot_Plated, F.Cu at (38.6, 24.0)
- added H3: MountingHole, 4ms_Faceplate:Faceplate_Rail_Mount_Slot_Plated, F.Cu at (104.5, 24.0)
- added H4: MountingHole, 4ms_Faceplate:Faceplate_Rail_Mount_Slot_Plated, F.Cu at (38.6, 146.5)
- added H5: MountingHole, 4ms_Faceplate:Faceplate_Rail_Mount_Slot_Plated, F.Cu at (104.5, 146.5)

Commit message: sizing, remove SW label
Parts:
- moved J10 3.01 mm to (90.4, 126.6)
- moved J5 3.00 mm to (39.2, 126.7)
- moved J6 3.00 mm to (49.9, 126.7)
- moved J7 3.00 mm to (60.5, 126.7)
- moved J8 3.00 mm to (71.2, 126.7)
- moved TP13 3.00 mm to (102.1, 126.1)
- moved H2 2.50 mm to (38.6, 21.5)
- moved H3 2.50 mm to (104.5, 21.5)
- moved H4 2.50 mm to (38.6, 144.0)
- moved H5 2.50 mm to (104.5, 144.0)
- moved C60 1.10 mm to (79.1, 41.0)
Connections:
- net /Power/SW renamed Net-(U4-SW)
Routing:
- net ADC3: track 129.1 -> 126.2 mm
- net /Outs/Out Pair 3/OP1_OUT: track 83.0 -> 80.7 mm
- net /Outs/Out Pair 4/OP1_OUT: track 80.5 -> 78.5 mm
- net /Outs/Out Pair 4/OP2_OUT: track 81.1 -> 79.9 mm
- net /Outs/Out Pair 3/OP2_OUT: track 74.3 -> 73.1 mm
- net +12V: track 341.4 -> 340.7 mm
Other:
- board text added: "Cut teensy power trace"
- board text added: "DC Interface Board Rev 1.0 Dan Lewis contact@danlewis.dev Alex Sludds alexsludds@gmail.com"

Commit message: Generated gerbers for boards
Parts:
- removed C10: 22uF_0805_6.3V, 4ms_Capacitor:C_0805
- removed C11: 10uF_0603_10V, 4ms_Capacitor:C_0603
- removed C12, C7, C9: 0.1uF_0603_16V, 4ms_Capacitor:C_0603
- removed C56: 22uF, 4ms_Capacitor:C_0805
- removed C57: 0.1uF, 4ms_Capacitor:C_0603
- removed C58: 47pF, 4ms_Capacitor:C_0603
- removed C59: 22uF, 4ms_Capacitor:C_0603
- removed C60: 10uF, 4ms_Capacitor:C_0603
- removed C61: 47uF, 4ms_Capacitor:CP_Elec_5x5.3
- removed C8: 22uF_0805_25V, 4ms_Capacitor:C_0805
- removed L1, L3: 15uH, 4ms_Inductor:COIL_5040
- removed L2: 4.7uH_1.2A_40xx, Inductor_SMD:L_Taiyo-Yuden_NR-40xx
- removed R1, R56: 100k, 4ms_Resistor:R_0603
- removed R2, R57: 75k, 4ms_Resistor:R_0603
- removed R3, R58: 40.2k, 4ms_Resistor:R_0603
- removed R4, R59: 7.68k, 4ms_Resistor:R_0603
- removed R5: 100k_0603, 4ms_Resistor:R_0603
- removed R6: 33.2k_0603, 4ms_Resistor:R_0603
- removed R7: 10k_0603, 4ms_Resistor:R_0603
- removed U9: AP65211A, 4ms_Package_SOT:TSOT-23-6
- added U10: NCP1117-5.0_SOT223, Package_TO_SOT_SMD:SOT-223-3_TabPin2, F.Cu at (90.6, 84.8)
- C1: value 22uF -> 10uF_0805_25V
- C2: value 0.1uF -> 10uF_0603_10V
- C3: value 47pF -> 10uF_0805_25V; footprint 4ms_Capacitor:C_0603 -> 4ms_Capacitor:C_0805
- C4: value 22uF -> 10uF_0603_10V
- C5: value 10uF -> 10uF_0805_25V; footprint 4ms_Capacitor:C_0603 -> 4ms_Capacitor:C_0805
- C6: value 47uF -> 10uF_0603_10V; footprint 4ms_Capacitor:CP_Elec_5x5.3 -> 4ms_Capacitor:C_0603
- U3: value AP65211A -> NCP1117-3.3_SOT223; footprint 4ms_Package_SOT:TSOT-23-6 -> Package_TO_SOT_SMD:SOT-223-3_TabPin2
- U4: value AP62200TWU-7 -> NCP1117-5.0_SOT223; footprint 4ms_Package_SOT:TSOT-23-6 -> Package_TO_SOT_SMD:SOT-223-3_TabPin2
- moved C4 51.3 mm to (82.6, 34.6), turned to 0 degrees
- moved C5 40.1 mm to (82.8, 46.6), turned to 0 degrees
- moved C6 25.7 mm to (91.6, 56.0), turned to 0 degrees
- moved U4 24.0 mm to (82.8, 40.5)
- moved U3 23.5 mm to (91.5, 62.3)
- moved C3 23.0 mm to (91.8, 67.6), turned to 0 degrees
- moved C2 7.79 mm to (94.0, 79.6)
- moved C1 5.51 mm to (90.8, 91.0), turned to 0 degrees
Connections:
- C2 pad 1: Net-(U3-SW) -> AVDD
- C2 pad 2: Net-(U3-BST) -> AVSS
- C3 pad 1: Net-(C3-Pad1) -> +12V
- C3 pad 2: AVDD -> DVSS
- C4 pad 1: AVDD -> TEENSY_5V
- C4 pad 2: AVSS -> DVSS
- C5 pad 1: AVDD -> +12V
- C5 pad 2: AVSS -> DVSS
- C6 pad 1: AVDD -> TVDD
- C6 pad 2: AVSS -> DVSS
- U3 pad 1: AVSS -> DVSS
- U3 pad 2: Net-(U3-SW) -> TVDD
- U4 pad 2: Net-(U4-SW) -> TEENSY_5V
Routing:
- net AVSS: track 223.3 -> 192.1 mm, vias 75 -> 80
- net +12V: track 340.7 -> 310.0 mm, vias 12 -> 10
- net Net-(U4-SW): track 19.7 -> 0.00 mm
- net Net-(U9-SW): track 17.6 -> 0.00 mm, vias 2 -> 0
- net Net-(U3-SW): track 14.4 -> 0.00 mm
- net DVSS: track 35.8 -> 24.9 mm, vias 15 -> 24
- net TEENSY_5V: track 74.0 -> 63.4 mm
- net Net-(U3-EN): track 9.94 -> 0.00 mm, vias 2 -> 0
- net Net-(C58-Pad1): track 9.53 -> 0.00 mm
- net Net-(U4-FB): track 9.42 -> 0.00 mm
- net Net-(C3-Pad1): track 9.38 -> 0.00 mm
- net Net-(U9-EN): track 8.61 -> 0.00 mm
- net Net-(U4-BST): track 7.11 -> 0.00 mm
- net TVDD: track 104.9 -> 111.2 mm, vias 4 -> 2
- net Net-(U4-EN): track 5.40 -> 0.00 mm
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
Commit message: dc interface
Routing:
- net ADC3: track 126.2 -> 124.7 mm
Changed lines of the file:
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@@
 	)
 	(segment
-		(start 62.462 31.918)
-		(end 69.618 31.918)
+		(start 71.5 33.8)
+		(end 71.5 37.4)
 		(width 0.2)
 		(layer "B.Cu")
@@
 	)
 	(segment
-		(start 72.1 36.91985)
-		(end 72.334315 37.154164)
+		(start 62.462 31.918)
+		(end 69.618 31.918)
 		(width 0.2)
 		(layer "B.Cu")
@@
 	)
 	(segment
-		(start 72.472164 37.292014)
+		(start 72.472164 38.372164)
 		(end 72.472164 59.572164)
 		(width 0.2)
@@
 	)
 	(segment
-		(start 72.1 35.18015)
-		(end 72.1 36.91985)
+		(start 71.5 37.4)
+		(end 72.472164 38.372164)
 		(width 0.2)
 		(layer "B.Cu")
@@
 	)
 	(segment
-		(start 61.46 32.92)
-		(end 62.462 31.918)
+		(start 69.618 31.918)
+		(end 71.5 33.8)
 		(width 0.2)
 		(layer "B.Cu")
@@
 	)
 	(segment
-		(start 72.472164 34.807986)
-		(end 72.1 35.18015)
-		(width 0.2)
-		(layer "B.Cu")
-		(net 30)
-	)
-	(segment
-		(start 72.472164 34.772164)
-		(end 72.472164 34.807986)
-		(width 0.2)
-		(layer "B.Cu")
-		(net 30)
-	)
-	(segment
-		(start 69.618 31.918)
-		(end 72.472164 34.772164)
-		(width 0.2)
-		(layer "B.Cu")
-		(net 30)
-	)
-	(segment
-		(start 72.334315 37.154164)
-		(end 72.472164 37.292014)
+		(start 61.46 32.92)
+		(end 62.462 31.918)
 		(width 0.2)
 		(layer "B.Cu")
@@
 	)
 	(segment
+		(start 97.85 59.15)
+		(end 94.7 62.3)
+		(width 0.5)
+		(layer "F.Cu")
+		(net 90)
+	)
+	(segment
 		(start 106.8 60)
 		(end 104.25 62.55)
@@
 	)
 	(segment
-		(start 57.950756 58.599244)
-		(end 55.2544 58.599244)
-		(width 0.2)
+		(start 102.325 61.475)
+		(end 100 59.15)
+		(width 0.5)
 		(layer "F.Cu")
 		(net 90)
 	)
 	(segment
-		(start 100 59.15)
-		(end 97.6 59.15)
-		(width 0.5)
+		(start 57.950756 58.599244)
+		(end 55.2544 58.599244)
+		(width 0.2)
 		(layer "F.Cu")
 		(net 90)
@@
 	)
 	(segment
-		(start 94.7 62.3)
-		(end 97.6 59.4)
-		(width 0.5)
-		(layer "F.Cu")
-		(net 90)
-	)
-	(segment
 		(start 103.4 63.6)
 		(end 103.4 62.55)
@@
 	)
 	(segment
-		(start 97.6 59.4)
-		(end 97.6 59.15)
+		(start 100 59.15)
+		(end 97.85 59.15)
 		(width 0.5)
 		(layer "F.Cu")
@@
 	)
 	(segment
-		(start 102.325 61.475)
-		(end 100 59.15)
-		(width 0.5)
-		(layer "F.Cu")
-		(net 90)
-	)
-	(segment
 		(start 101.4 68.35)
 		(end 101.6 68.55)
@@
 	)
 	(segment
-		(start 90.6 121.4402)
-		(end 97.4402 121.4402)
-		(width 0.2)
-		(layer "B.Cu")
-		(net 100)
-	)
-	(segment
-		(start 90.9 77.434314)
-		(end 90.9 105.703737)
-		(width 0.2)
-		(layer "B.Cu")
-		(net 100)
-	)
-	(segment
-		(start 73 37.254164)
+		(start 73 38.2)
 		(end 73 59.534314)
 		(width 0.2)
@@
 	)
 	(segment
-		(start 73 32.445836)
-		(end 73 34.845836)
+		(start 90.6 121.4402)
+		(end 97.4402 121.4402)
 		(width 0.2)
 		(layer "B.Cu")
@@
 	)
 	(segment
-		(start 72.072164 31.518)
-		(end 73 32.445836)
+		(start 60.322 31.518)
+		(end 70.218 31.518)
 		(width 0.2)
 		(layer "B.Cu")
@@
 	(segment
 		(start 91.6652 120.175)
-		(end 91.6652 106.468937)
+		(end 90.4 121.4402)
 		(width 0.2)
 		(layer "B.Cu")
@@
 	)
 	(segment
-		(start 73 34.845836)
-		(end 72.5 35.345836)
+		(start 73 59.534314)
+		(end 90.9 77.434314)
 		(width 0.2)
 		(layer "B.Cu")
@@
 	)
 	(segment
-		(start 73 59.534314)
-		(end 90.9 77.434314)
+		(start 91.6652 106.468937)
+		(end 91.6652 120.175)
 		(width 0.2)
 		(layer "B.Cu")
@@
 	)
 	(segment
-		(start 72.5 35.345836)
-		(end 72.5 36.754164)
+		(start 90.9 77.434314)
+		(end 90.9 105.703737)
 		(width 0.2)
 		(layer "B.Cu")
@@
 	)
 	(segment
-		(start 72.5 36.754164)
-		(end 73 37.254164)
+		(start 72 33.3)
+		(end 72 37.2)
 		(width 0.2)
 		(layer "B.Cu")
@@
 	)
 	(segment
-		(start 90.4 121.4402)
-		(end 91.6652 120.175)
+		(start 70.218 31.518)
+		(end 72 33.3)
 		(width 0.2)
 		(layer "B.Cu")
@@
 	)
 	(segment
-		(start 60.322 31.518)
-		(end 72.072164 31.518)
+		(start 72 37.2)
+		(end 73 38.2)
 		(width 0.2)
 		(layer "B.Cu")
@@
 		(min_thickness 0.25)
 		(filled_areas_thickness no)
-		(fill
+		(fill yes
 			(thermal_gap 0.5)
 			(thermal_bridge_width 0.5)
@@
 		(min_thickness 0.25)
 		(filled_areas_thickness no)
-		(fill
+		(fill yes
 			(thermal_gap 0.5)
 			(thermal_bridge_width 0.5)
