File: switch_sequencer/power_attenuverters.kicad_sch (KiCad schematic)
At the start: 0 parts

Commit message: Updated schematic of sample and hold, attenuveters, sequential switch
Parts:
- added C13: 0.1uF_0805_50V, 4ms_Capacitor:C_0805, symbol 4ms_Capacitor:0.1uF_0805_50V
- added C14, C15: 10uF_0603_10V, 4ms_Capacitor:C_0603, symbol 4ms_Capacitor:10uF_0603_10V
- added C16: 1uF_0603_25V, 4ms_Capacitor:C_0603, symbol 4ms_Capacitor:1uF_0603_25V
- added C17: 10nF_0603_25V, 4ms_Capacitor:C_0603, symbol 4ms_Capacitor:10nF_0603_25V
- added J24: Eurorack_Power_10pin_Shrouded, 4ms_Connector:Pins_2x05_2.54mm_TH_EurorackPower_Shrouded, symbol 4ms_Connector:Eurorack_Power_10pin_Shrouded
- added U11: LD1117S50TR_SOT223, Package_TO_SOT_SMD:SOT-223-3_TabPin2, symbol Regulator_Linear:LD1117S50TR_SOT223
- added U14: LT1964-5, Package_TO_SOT_SMD:TSOT-23-5, symbol Regulator_Linear:LT1964-5
Connections:
- new net: C17.1, U14.3 (BYP)
- new net +12V: C13.1, J24.10 (+12V), J24.9 (+12V), U11.3 (VI)
- new net -12VA: C16.1, J24.1 (-12V), J24.2 (-12V), U14.2 (VIN), U14.4 (~{SHDN})
- new net 5V: C14.1, U11.2 (VO)
- new net GND: C13.2, C14.2, C15.1, C16.2, J24.3 (GND), J24.4 (GND), J24.5 (GND), J24.6 (GND), J24.7 (GND), J24.8 (GND), U11.1 (GND), U14.1 (GND)
- new net minus_5V: C15.2, C17.2, U14.5 (VOUT)
