File: switch_sequencer/power_sequencer_switch.kicad_sch (KiCad schematic)
At the start: 12 parts, among them J12 Eurorack_Power_10pin_Shrouded, U3 AP62200TWU-7

Commit message: Updated schematic of sample and hold, attenuveters, sequential switch
Parts:
- added C11: 0.1uF_0805_50V, 4ms_Capacitor:C_0805, symbol 4ms_Capacitor:0.1uF_0805_50V
- added C12: 10uF_0603_10V, 4ms_Capacitor:C_0603, symbol 4ms_Capacitor:10uF_0603_10V
- added U9: LD1117S50TR_SOT223, Package_TO_SOT_SMD:SOT-223-3_TabPin2, symbol Regulator_Linear:LD1117S50TR_SOT223
- renumbered J12 to J13
Connections:
- net +12V: now also C11.1, U9.3 (VI)
- net GND: now also C11.2, C12.2, U9.1 (GND)
- new net 5V: C12.1, U9.2 (VO)
