File: switch_sequencer/two_attenuverters.kicad_sch (KiCad schematic)
At the start: 0 parts

Commit message: Updated schematic of sample and hold, attenuveters, sequential switch
Parts:
- added Attenuverter1, Attenuverter2, Attenuverter3, Attenuverter4, Attenuverter5, Attenuverter6, Attenuverter7, Attenuverter8: 100k, Eurocad:Alpha9mmPot, symbol Device:R_Potentiometer
- added J22, J23, J26, J27, J28, J29, J30, J31, J32, J33, J34, J35, J36, J37, J38, J39: 3.5mm_Mono_Switched_sm, 4ms_Jack:EighthInch_PJ398SM, symbol 4ms_Jack:3.5mm_Mono_Switched_sm
- added J25, J40: Conn_01x03, 4ms_Connector:Pins_1x03_2.54mm_TH, symbol 4ms_Connector:Conn_01x03
- added R10, R11, R12, R13, R14, R15, R16, R17, R18, R19, R4, R5, R6, R7, R8, R9: 100k, Resistor_THT:R_Axial_DIN0207_L6.3mm_D2.5mm_P10.16mm_Horizontal, symbol Device:R
- added U10, U11, U12, U13: LM358, LM358PE3:DIP794W45P254L959H508Q8, symbol Amplifier_Operational:LM358
Connections:
- new net: J23.1 (SIG), R5.2, U10.1
- new net: Attenuverter5.3, J32.1 (SIG), R12.1
- new net: R12.2, R16.1, U13.6 (-)
- new net: Attenuverter2.2, U10.5 (+)
- new net: R6.2, R7.1, U10.6 (-)
- new net: J27.1 (SIG), R7.2, U10.7
- new net: J36.1 (SIG), R16.2, U13.7
- new net: Attenuverter5.2, U13.5 (+)
- new net: R8.2, R9.1, U11.2 (-)
- new net: J29.1 (SIG), R9.2, U11.1
- new net: J37.1 (SIG), R17.2, U12.7
- new net: Attenuverter7.2, U13.3 (+)
- new net: Attenuverter7.3, J34.1 (SIG), R14.1
- new net: R10.2, R11.1, U11.6 (-)
- new net: J31.1 (SIG), R11.2, U11.7
- new net: Attenuverter1.2, U10.3 (+)
- new net: Attenuverter1.3, J22.1 (SIG), R4.1
- new net: Attenuverter4.3, J30.1 (SIG), R10.1
- new net: R4.2, R5.1, U10.2 (-)
- new net: Attenuverter6.2, U12.5 (+)
- new net: Attenuverter6.3, J33.1 (SIG), R13.1
- new net: Attenuverter2.3, J26.1 (SIG), R6.1
- new net: R14.2, R18.1, U13.2 (-)
- new net: J38.1 (SIG), R18.2, U13.1
- new net: Attenuverter8.3, J35.1 (SIG), R15.1
- new net: R15.2, R19.1, U12.2 (-)
- new net: Attenuverter4.2, U11.5 (+)
- new net: R13.2, R17.1, U12.6 (-)
- new net: J39.1 (SIG), R19.2, U12.1
- new net: Attenuverter3.3, J28.1 (SIG), R8.1
- new net: Attenuverter8.2, U12.3 (+)
- new net: Attenuverter3.2, U11.3 (+)
- new net +12V: J25.1 (Pin_1)
- new net -12VA: J40.1 (Pin_1)
- new net 5V: J25.3 (Pin_3)
- new net GND: Attenuverter1.1, Attenuverter2.1, Attenuverter3.1, Attenuverter4.1, Attenuverter5.1, Attenuverter6.1, Attenuverter7.1, Attenuverter8.1
- new net GNDA: J22.2 (SHEILD), J22.3 (SW), J23.2 (SHEILD), J23.3 (SW), J26.2 (SHEILD), J26.3 (SW), J27.2 (SHEILD), J27.3 (SW), J28.2 (SHEILD), J28.3 (SW), J29.2 (SHEILD), J29.3 (SW), J30.2 (SHEILD), J30.3 (SW), J31.2 (SHEILD), J31.3 (SW), J32.2 (SHEILD), J32.3 (SW), J33.2 (SHEILD), J33.3 (SW), J34.2 (SHEILD), J34.3 (SW), J35.2 (SHEILD), J35.3 (SW), J36.2 (SHEILD), J36.3 (SW), J37.2 (SHEILD), J37.3 (SW), J38.2 (SHEILD), J38.3 (SW), J39.2 (SHEILD), J39.3 (SW)
- new net minus_5V: J40.3 (Pin_3)
- new net op_amp_negative_supply: J40.2 (Pin_2), U10.4 (V-), U11.4 (V-), U12.4 (V-), U13.4 (V-)
- new net op_amp_positive_supply: J25.2 (Pin_2), U10.8 (V+), U11.8 (V+), U12.8 (V+), U13.8 (V+)
