File: switch_sequencer/switch_sequencer/i_o_sequencer_switch.kicad_sch (KiCad schematic)
At the start: 13 parts, among them J1 Conn_01x09, J10 3.5mm_Mono_Switched_sm, J11 3.5mm_Mono_Switched_sm, J2 Conn_01x09, J20 3.5mm_Mono_Switched_sm, J21 3.5mm_Mono_Switched_sm, J3 3.5mm_Mono_Switched_sm, J4 3.5mm_Mono_Switched_sm, J5 3.5mm_Mono_Switched_sm, J6 3.5mm_Mono_Switched_sm, J7 3.5mm_Mono_Switched_sm, J8 3.5mm_Mono_Switched_sm, J9 3.5mm_Mono_Switched_sm

Commit message: Reformated folder structure. Finished layout of sample and hold.
Parts:
- renumbered J7 to J10, J8 to J11, J9 to J12, J10 to J13, J11 to J4, J4 to J5, J20 to J6, J5 to J7, J21 to J8, J6 to J9

Commit message: sequential switch wip
Parts:
- removed J10, J11, J12, J13, J3, J4, J5, J6, J7, J8, J9: 3.5mm_Mono_Switched_sm, 4ms_Jack:EighthInch_PJ398SM, symbol 4ms_Jack:3.5mm_Mono_Switched_sm
