File: switch_sequencer/switch_sequencer/led.kicad_sch (KiCad schematic)
At the start: 2 parts

Commit message: sequential swtich more wip
Parts:
- removed C14: 100nF_0402_16V, 4ms_Capacitor:C_0402, symbol 4ms_Capacitor:100nF_0402_16V
- added C15: 100nF_0402_16V, 4ms_Capacitor:C_0402, symbol 4ms_Capacitor:100nF_0402_16V
- renumbered D12 to D18
Connections:
- net 5V: now also C15.1
- net GND: now also C15.2
Changed lines of the file:
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@@
 		(on_board yes)
 		(dnp no)
-		(property "Reference" "#PWR069"
+		(property "Reference" "#PWR045"
 			(at 100.33 97.79 0)
 			(effects
@@
 				(path "/1090b42d-0526-4901-ae26-1a4493d10820/4c22d006-f8e0-4fe5-9164-b59b12367ed8/ff53a658-11dc-478f-9769-67012b38ead8/d8422442-063e-469c-9c55-c5e9b5255364"
 					(reference "#PWR076")
+					(unit 1)
+				)
+			)
+		)
+	)
+	(symbol
+		(lib_id "4ms_Power-symbol:GND")
+		(at 100.33 73.66 0)
+		(unit 1)
+		(exclude_from_sim no)
+		(in_bom yes)
+		(on_board yes)
+		(dnp no)
+		(property "Reference" "#PWR041"
+			(at 100.33 80.01 0)
+			(effects
+				(font
+					(size 1.27 1.27)
+				)
+				(hide yes)
+			)
+		)
+		(property "Value" "GND"
+			(at 100.33 77.47 0)
+			(effects
+				(font
+					(size 1.27 1.27)
+				)
+			)
+		)
+		(property "Footprint" ""
+			(at 100.33 73.66 0)
+			(effects
+				(font
+					(size 1.27 1.27)
+				)
+				(hide yes)
+			)
+		)
+		(property "Datasheet" ""
+			(at 100.33 73.66 0)
+			(effects
+				(font
+					(size 1.27 1.27)
+				)
+				(hide yes)
+			)
+		)
+		(property "Description" ""
+			(at 100.33 73.66 0)
+			(effects
+				(font
+					(size 1.27 1.27)
+				)
+				(hide yes)
+			)
+		)
+		(pin "1"
+		)
+		(instances
+			(project "switch_sequencer"
+				(path "/1090b42d-0526-4901-ae26-1a4493d10820/62063eaf-8a8e-4b69-9d16-9268e74da748"
+					(reference "#PWR041")
+					(unit 1)
+				)
+				(path "/1090b42d-0526-4901-ae26-1a4493d10820/7dc0a39b-b136-4016-be0c-c023d8387e8a"
+					(reference "#PWR04")
+					(unit 1)
+				)
+				(path "/1090b42d-0526-4901-ae26-1a4493d10820/4c22d006-f8e0-4fe5-9164-b59b12367ed8/3b32ef6f-f7de-4ddd-97a9-3d5452522cd1/d8422442-063e-469c-9c55-c5e9b5255364"
+					(reference "#PWR068")
+					(unit 1)
+				)
+				(path "/1090b42d-0526-4901-ae26-1a4493d10820/4c22d006-f8e0-4fe5-9164-b59b12367ed8/5043bc26-4ce4-47be-bac8-88b06297739f/d8422442-063e-469c-9c55-c5e9b5255364"
+					(reference "#PWR082")
+					(unit 1)
+				)
+				(path "/1090b42d-0526-4901-ae26-1a4493d10820/4c22d006-f8e0-4fe5-9164-b59b12367ed8/56a49501-ca12-4951-9aa9-3235726846b6/d8422442-063e-469c-9c55-c5e9b5255364"
+					(reference "#PWR035")
+					(unit 1)
+				)
+				(path "/1090b42d-0526-4901-ae26-1a4493d10820/4c22d006-f8e0-4fe5-9164-b59b12367ed8/7e64556a-f431-4fba-8c1d-6e9af7db61e9/d8422442-063e-469c-9c55-c5e9b5255364"
+					(reference "#PWR061")
+					(unit 1)
+				)
+				(path "/1090b42d-0526-4901-ae26-1a4493d10820/4c22d006-f8e0-4fe5-9164-b59b12367ed8/a947920c-59f2-438b-89ba-8e48f95d6dbc/d8422442-063e-469c-9c55-c5e9b5255364"
+					(reference "#PWR054")
+					(unit 1)
+				)
+				(path "/1090b42d-0526-4901-ae26-1a4493d10820/4c22d006-f8e0-4fe5-9164-b59b12367ed8/ab8d2706-56a5-4587-b9ef-c598dc5bc3f9/d8422442-063e-469c-9c55-c5e9b5255364"
+					(reference "#PWR011")
+					(unit 1)
+				)
+				(path "/1090b42d-0526-4901-ae26-1a4493d10820/4c22d006-f8e0-4fe5-9164-b59b12367ed8/f6bf03c5-1acc-4c33-9962-bfdc3f3d33ad/d8422442-063e-469c-9c55-c5e9b5255364"
+					(reference "#PWR018")
+					(unit 1)
+				)
+				(path "/1090b42d-0526-4901-ae26-1a4493d10820/4c22d006-f8e0-4fe5-9164-b59b12367ed8/ff53a658-11dc-478f-9769-67012b38ead8/d8422442-063e-469c-9c55-c5e9b5255364"
+					(reference "#PWR075")
 					(unit 1)
 				)
@@
 		(dnp no)
 		(fields_autoplaced yes)
-		(property "Reference" "C14"
+		(property "Reference" "C15"
 			(at 102.87 87.6362 0)
 			(effects
@@
 			(project "switch_sequencer"
 				(path "/1090b42d-0526-4901-ae26-1a4493d10820/62063eaf-8a8e-4b69-9d16-9268e74da748"
-					(reference "C3")
+					(reference "C24")
 					(unit 1)
 				)
 				(path "/1090b42d-0526-4901-ae26-1a4493d10820/7dc0a39b-b136-4016-be0c-c023d8387e8a"
-					(reference "C4")
+					(reference "C15")
 					(unit 1)
 				)
 				(path "/1090b42d-0526-4901-ae26-1a4493d10820/4c22d006-f8e0-4fe5-9164-b59b12367ed8/3b32ef6f-f7de-4ddd-97a9-3d5452522cd1/d8422442-063e-469c-9c55-c5e9b5255364"
-					(reference "C14")
+					(reference "C21")
 					(unit 1)
 				)
 				(path "/1090b42d-0526-4901-ae26-1a4493d10820/4c22d006-f8e0-4fe5-9164-b59b12367ed8/5043bc26-4ce4-47be-bac8-88b06297739f/d8422442-063e-469c-9c55-c5e9b5255364"
+					(reference "C23")
+					(unit 1)
+				)
+				(path "/1090b42d-0526-4901-ae26-1a4493d10820/4c22d006-f8e0-4fe5-9164-b59b12367ed8/56a49501-ca12-4951-9aa9-3235726846b6/d8422442-063e-469c-9c55-c5e9b5255364"
+					(reference "C18")
+					(unit 1)
+				)
+				(path "/1090b42d-0526-4901-ae26-1a4493d10820/4c22d006-f8e0-4fe5-9164-b59b12367ed8/7e64556a-f431-4fba-8c1d-6e9af7db61e9/d8422442-063e-469c-9c55-c5e9b5255364"
+					(reference "C20")
+					(unit 1)
+				)
+				(path "/1090b42d-0526-4901-ae26-1a4493d10820/4c22d006-f8e0-4fe5-9164-b59b12367ed8/a947920c-59f2-438b-89ba-8e48f95d6dbc/d8422442-063e-469c-9c55-c5e9b5255364"
+					(reference "C19")
+					(unit 1)
+				)
+				(path "/1090b42d-0526-4901-ae26-1a4493d10820/4c22d006-f8e0-4fe5-9164-b59b12367ed8/ab8d2706-56a5-4587-b9ef-c598dc5bc3f9/d8422442-063e-469c-9c55-c5e9b5255364"
 					(reference "C16")
 					(unit 1)
 				)
-				(path "/1090b42d-0526-4901-ae26-1a4493d10820/4c22d006-f8e0-4fe5-9164-b59b12367ed8/56a49501-ca12-4951-9aa9-3235726846b6/d8422442-063e-469c-9c55-c5e9b5255364"
-					(reference "C11")
-					(unit 1)
-				)
-				(path "/1090b42d-0526-4901-ae26-1a4493d10820/4c22d006-f8e0-4fe5-9164-b59b12367ed8/7e64556a-f431-4fba-8c1d-6e9af7db61e9/d8422442-063e-469c-9c55-c5e9b5255364"
-					(reference "C13")
-					(unit 1)
-				)
-				(path "/1090b42d-0526-4901-ae26-1a4493d10820/4c22d006-f8e0-4fe5-9164-b59b12367ed8/a947920c-59f2-438b-89ba-8e48f95d6dbc/d8422442-063e-469c-9c55-c5e9b5255364"
-					(reference "C12")
-					(unit 1)
-				)
-				(path "/1090b42d-0526-4901-ae26-1a4493d10820/4c22d006-f8e0-4fe5-9164-b59b12367ed8/ab8d2706-56a5-4587-b9ef-c598dc5bc3f9/d8422442-063e-469c-9c55-c5e9b5255364"
-					(reference "C9")
-					(unit 1)
-				)
 				(path "/1090b42d-0526-4901-ae26-1a4493d10820/4c22d006-f8e0-4fe5-9164-b59b12367ed8/f6bf03c5-1acc-4c33-9962-bfdc3f3d33ad/d8422442-063e-469c-9c55-c5e9b5255364"
-					(reference "C10")
+					(reference "C17")
 					(unit 1)
 				)
 				(path "/1090b42d-0526-4901-ae26-1a4493d10820/4c22d006-f8e0-4fe5-9164-b59b12367ed8/ff53a658-11dc-478f-9769-67012b38ead8/d8422442-063e-469c-9c55-c5e9b5255364"
-					(reference "C15")
-					(unit 1)
-				)
-			)
-		)
-	)
-	(symbol
-		(lib_id "4ms_Power-symbol:GND")
-		(at 100.33 73.66 0)
-		(unit 1)
-		(exclude_from_sim no)
-		(in_bom yes)
-		(on_board yes)
-		(dnp no)
-		(property "Reference" "#PWR068"
-			(at 100.33 80.01 0)
-			(effects
-				(font
-					(size 1.27 1.27)
-				)
-				(hide yes)
-			)
-		)
-		(property "Value" "GND"
-			(at 100.33 77.47 0)
-			(effects
-				(font
-					(size 1.27 1.27)
-				)
-			)
-		)
-		(property "Footprint" ""
-			(at 100.33 73.66 0)
-			(effects
-				(font
-					(size 1.27 1.27)
-				)
-				(hide yes)
-			)
-		)
-		(property "Datasheet" ""
-			(at 100.33 73.66 0)
-			(effects
-				(font
-					(size 1.27 1.27)
-				)
-				(hide yes)
-			)
-		)
-		(property "Description" ""
-			(at 100.33 73.66 0)
-			(effects
-				(font
-					(size 1.27 1.27)
-				)
-				(hide yes)
-			)
-		)
-		(pin "1"
-		)
-		(instances
-			(project "switch_sequencer"
-				(path "/1090b42d-0526-4901-ae26-1a4493d10820/62063eaf-8a8e-4b69-9d16-9268e74da748"
-					(reference "#PWR041")
-					(unit 1)
-				)
-				(path "/1090b42d-0526-4901-ae26-1a4493d10820/7dc0a39b-b136-4016-be0c-c023d8387e8a"
-					(reference "#PWR04")
-					(unit 1)
-				)
-				(path "/1090b42d-0526-4901-ae26-1a4493d10820/4c22d006-f8e0-4fe5-9164-b59b12367ed8/3b32ef6f-f7de-4ddd-97a9-3d5452522cd1/d8422442-063e-469c-9c55-c5e9b5255364"
-					(reference "#PWR068")
-					(unit 1)
-				)
-				(path "/1090b42d-0526-4901-ae26-1a4493d10820/4c22d006-f8e0-4fe5-9164-b59b12367ed8/5043bc26-4ce4-47be-bac8-88b06297739f/d8422442-063e-469c-9c55-c5e9b5255364"
-					(reference "#PWR082")
-					(unit 1)
-				)
-				(path "/1090b42d-0526-4901-ae26-1a4493d10820/4c22d006-f8e0-4fe5-9164-b59b12367ed8/56a49501-ca12-4951-9aa9-3235726846b6/d8422442-063e-469c-9c55-c5e9b5255364"
-					(reference "#PWR035")
-					(unit 1)
-				)
-				(path "/1090b42d-0526-4901-ae26-1a4493d10820/4c22d006-f8e0-4fe5-9164-b59b12367ed8/7e64556a-f431-4fba-8c1d-6e9af7db61e9/d8422442-063e-469c-9c55-c5e9b5255364"
-					(reference "#PWR061")
-					(unit 1)
-				)
-				(path "/1090b42d-0526-4901-ae26-1a4493d10820/4c22d006-f8e0-4fe5-9164-b59b12367ed8/a947920c-59f2-438b-89ba-8e48f95d6dbc/d8422442-063e-469c-9c55-c5e9b5255364"
-					(reference "#PWR054")
-					(unit 1)
-				)
-				(path "/1090b42d-0526-4901-ae26-1a4493d10820/4c22d006-f8e0-4fe5-9164-b59b12367ed8/ab8d2706-56a5-4587-b9ef-c598dc5bc3f9/d8422442-063e-469c-9c55-c5e9b5255364"
-					(reference "#PWR011")
-					(unit 1)
-				)
-				(path "/1090b42d-0526-4901-ae26-1a4493d10820/4c22d006-f8e0-4fe5-9164-b59b12367ed8/f6bf03c5-1acc-4c33-9962-bfdc3f3d33ad/d8422442-063e-469c-9c55-c5e9b5255364"
-					(reference "#PWR018")
-					(unit 1)
-				)
-				(path "/1090b42d-0526-4901-ae26-1a4493d10820/4c22d006-f8e0-4fe5-9164-b59b12367ed8/ff53a658-11dc-478f-9769-67012b38ead8/d8422442-063e-469c-9c55-c5e9b5255364"
-					(reference "#PWR075")
+					(reference "C22")
 					(unit 1)
 				)
@@
 		(on_board yes)
 		(dnp no)
-		(property "Reference" "D12"
+		(property "Reference" "D18"
 			(at 100.33 48.514 0)
 			(effects

Commit message: sequential switch finished
Parts:
- renumbered C15 to C25, D18 to D20
Changed lines of the file:
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@@
 		(on_board yes)
 		(dnp no)
-		(property "Reference" "#PWR045"
+		(property "Reference" "#PWR089"
 			(at 100.33 97.79 0)
 			(effects
@@
 		(on_board yes)
 		(dnp no)
-		(property "Reference" "#PWR041"
+		(property "Reference" "#PWR088"
 			(at 100.33 80.01 0)
 			(effects
@@
 		(dnp no)
 		(fields_autoplaced yes)
-		(property "Reference" "C15"
+		(property "Reference" "C25"
 			(at 102.87 87.6362 0)
 			(effects
@@
 		(on_board yes)
 		(dnp no)
-		(property "Reference" "D18"
+		(property "Reference" "D20"
 			(at 100.33 48.514 0)
 			(effects
