File: double_pendulum/power.kicad_sch (KiCad schematic)
At the start: 18 parts, among them J12 Eurorack_Power_16pin_Shrouded, U2 TL072, U3 TL072, U5 TL072, U6 LM7805_TO220

Commit message: double pendulum 4ms package path update
Parts:
- J12: footprint PCM_4ms_Connector:Pins_2x08_2.54mm_TH_EuroPower_Shrouded -> 4ms_Connector:Pins_2x05_2.54mm_TH_EurorackPower
- U2, U3, U5: footprint PCM_4ms_Package_SSOP:TSSOP-8_4.4x3mm_Pitch0.65mm -> 4ms_Package_SSOP:TSSOP-8_4.4x3mm_Pitch0.65mm
Changed lines of the file:
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@@
 			)
 		)
-		(property "Footprint" "PCM_4ms_Package_SSOP:TSSOP-8_4.4x3mm_Pitch0.65mm"
+		(property "Footprint" "4ms_Package_SSOP:TSSOP-8_4.4x3mm_Pitch0.65mm"
 			(at 46.99 95.25 0)
 			(effects
@@
 			)
 		)
-		(property "Footprint" "PCM_4ms_Connector:Pins_2x08_2.54mm_TH_EuroPower_Shrouded"
+		(property "Footprint" "4ms_Connector:Pins_2x05_2.54mm_TH_EurorackPower"
 			(at 44.45 52.07 0)
 			(effects
@@
 			)
 		)
-		(property "Footprint" "PCM_4ms_Package_SSOP:TSSOP-8_4.4x3mm_Pitch0.65mm"
+		(property "Footprint" "4ms_Package_SSOP:TSSOP-8_4.4x3mm_Pitch0.65mm"
 			(at 74.93 93.98 0)
 			(effects
@@
 			)
 		)
-		(property "Footprint" "PCM_4ms_Package_SSOP:TSSOP-8_4.4x3mm_Pitch0.65mm"
+		(property "Footprint" "4ms_Package_SSOP:TSSOP-8_4.4x3mm_Pitch0.65mm"
 			(at 59.69 95.25 0)
 			(effects

Commit message: Finished schematic and layout of the double pendulum
Parts:
- removed C1, C2: 0.33u, Capacitor_SMD:C_0805_2012Metric, symbol Device:C
- removed J12: Eurorack_Power_16pin_Shrouded, 4ms_Connector:Pins_2x05_2.54mm_TH_EurorackPower, symbol PCM_4ms_Connector:Eurorack_Power_16pin_Shrouded
- removed U2, U3, U5: TL072, 4ms_Package_SSOP:TSSOP-8_4.4x3mm_Pitch0.65mm, symbol PCM_4ms_IC:TL072
- removed U6: LM7805_TO220, Package_TO_SOT_THT:TO-220-3_Vertical, symbol Regulator_Linear:LM7805_TO220
- added C1: 0.1uF_0805_50V, Capacitor_SMD:C_0805_2012Metric, symbol 4ms_Capacitor:0.1uF_0805_50V
- added C2: 10uF_0603_10V, Capacitor_SMD:C_0805_2012Metric, symbol 4ms_Capacitor:10uF_0603_10V
- added J1: Eurorack_Power_10pin_Shrouded, 4ms_Connector:Pins_2x05_2.54mm_TH_EurorackPower_Shrouded, symbol 4ms_Connector:Eurorack_Power_10pin_Shrouded
- added U4: LD1117S50TR_SOT223, Package_TO_SOT_SMD:SOT-223-3_TabPin2, symbol Regulator_Linear:LD1117S50TR_SOT223
Connections:
- net 5V: now also C2.1, U4.2 (VO)
- net GND: now also C1.2, C2.2, J1.3 (GND), J1.4 (GND), J1.5 (GND), J1.6 (GND), J1.7 (GND), J1.8 (GND), U4.1 (GND)
- net 12V renamed +12V
- net +12V: now also C1.1, J1.10 (+12V), J1.9 (+12V), U4.3 (VI)
- new net -12VA: J1.1 (-12V), J1.2 (-12V)
- no-connect marks 8 -> 0
